Commit message: new hall_to_odom.py

File: my_robot_description/urdf/lidar.xacro (robot description, xacro)
@@ -1,10 +1,11 @@
 <?xml version="1.0"?>
 <robot xmlns:xacro="http://www.ros.org/wiki/xacro" >
-    <joint name="laser_joint" type="fixed">
+<!-- LIDAR 1 (back) -->
+    <joint name="laser_1_joint" type="fixed">
         <parent link="base_link"/>
-        <child link="laser_frame"/>
-        <origin xyz="-0.5 0 0.26" rpy="0 0 3.14159"/>
+        <child link="laser_1_frame"/>
+        <origin xyz="-0.48 -0.38 0.26" rpy="0 0 0"/>
     </joint>
-    <link name="laser_frame">
+    <link name="laser_1_frame">
         <visual>
             <geometry>
@@ -22,29 +23,79 @@
         </xacro:inertial_cylinder>
     </link>
-    <gazebo reference="laser_frame">
+    <gazebo reference="laser_1_frame">
         <material>Gazebo/Black</material>
-        <sensor name="laser" type="ray">
+        <sensor name="laser_1" type="ray">
             <pose> 0 0 0 0 0 0 </pose>
             <visualize>true</visualize>
-            <update_rate>10</update_rate>
+            <update_rate>20</update_rate>
             <ray>
                 <scan>
                     <horizontal>
                         <samples>270</samples>
-                        <min_angle>-1.745</min_angle>
-                        <max_angle>1.745</max_angle>
+                        <min_angle>-1.57</min_angle>
+                        <max_angle>3.14159</max_angle>
                     </horizontal>
                 </scan>
                 <range>
-                    <min>0.3</min>
+                    <min>0.1</min>
                     <max>20</max>
                 </range>
             </ray>
-            <plugin name="laser_controller" filename="libgazebo_ros_ray_sensor.so">
+            <plugin name="laser1_controller" filename="libgazebo_ros_ray_sensor.so">
                 <ros>
-                    <argument>~/out:=scan</argument>
+                    <remapping>~/out:=scan_1</remapping>
                 </ros>
                 <output_type>sensor_msgs/LaserScan</output_type>
-                <frame_name>laser_frame</frame_name>
+                <frame_name>laser_1_frame</frame_name>
+            </plugin>
+        </sensor>
+    </gazebo>
+<!-- LIDAR 2 (front) -->
+    <joint name="laser_2_joint" type="fixed">
+        <parent link="base_link"/>
+        <child link="laser_2_frame"/>
+        <origin xyz="0.48 0.38 0.26" rpy="0 0 3.14159"/>
+    </joint>
+    <link name="laser_2_frame">
+        <visual>
+            <geometry>
+                <cylinder radius="0.03" length="0.03"/>
+            </geometry>
+            <material name="black"/>
+        </visual>
+        <collision>
+            <geometry>
+                <cylinder radius="0.05" length="0.04"/>
+            </geometry>
+        </collision>
+        <xacro:inertial_cylinder mass="0.1" length="0.04" radius="0.05">
+            <origin xyz="0 0 0" rpy="0 0 0"/>
+        </xacro:inertial_cylinder>
+    </link>
+    <gazebo reference="laser_2_frame">
+        <material>Gazebo/Black</material>
+        <sensor name="laser_2" type="ray">
+            <pose> 0 0 0 0 0 0 </pose>
+            <visualize>true</visualize>
+            <update_rate>20</update_rate>
+            <ray>
+                <scan>
+                    <horizontal>
+                        <samples>270</samples>
+                        <min_angle>-1.57</min_angle>
+                        <max_angle>3.14159</max_angle>
+                    </horizontal>
+                </scan>
+                <range>
+                    <min>0.1</min>
+                    <max>20</max>
+                </range>
+            </ray>
+            <plugin name="laser2_controller" filename="libgazebo_ros_ray_sensor.so">
+                <ros>
+                    <remapping>~/out:=scan_2</remapping>
+                </ros>
+                <output_type>sensor_msgs/LaserScan</output_type>
+                <frame_name>laser_2_frame</frame_name>
             </plugin>
         </sensor>

File: my_robot_description/urdf/my_robot.xacro (robot description, xacro)
@@ -33,5 +33,5 @@
   <parent link="base_footprint"/>
   <child link="base_link"/>
-  <origin xyz="0 0 0" rpy="0 0 0"/>
+  <origin xyz="0 0 0" rpy="0 0 3.14159"/>
 </joint>
 <!-- RIGHT WHEEL LINK -->
